File: kairo/keyboard.kicad_pcb (KiCad board)
At the start: 2 copper layers, 1 part, among them U1 ProMicro

Commit message: 実装基盤図の更新
保存し忘れ
Parts:
- added SW1: SW_PUSH, BrownSugar_KBD:Kailh_Choc_V1_Hotswap_via, F.Cu at (89.8, 52.4)
